Commit message: Added lidar and camera alongwith color

File: catkin_ws/src/my_robot/urdf/my_robot.xacro (robot description, xacro)
@@ -36,4 +36,16 @@
 		</geometry>
 	</collision>
+	<visual name="back_caster_visual">
+		<origin xyz="-0.15 0 -0.05" rpy=" 0 0 0"/>
+		<geometry>
+			<sphere radius="0.05"/>
+		</geometry>
+	</visual>
+	<collision name="front_caster_collision">
+		<origin xyz="0.15 0 -0.05" rpy=" 0 0 0"/>
+		<geometry>
+			<sphere radius="0.0499"/>
+		</geometry>
+	</collision>
 	<visual name="front_caster_visual">
 		<origin xyz="0.15 0 -0.05" rpy=" 0 0 0"/>
@@ -43,3 +55,136 @@
 	</visual>
 	</link>
+	<link name="left_wheel">
+		<inertial>
+		<mass value="5.0"/>
+		<origin xyz="0 0 0" rpy="0 1.5707 1.5707"/>
+		<inertia
+			ixx="0.1" ixy="0" ixz="0"
+			iyy="0.1" iyz="0"
+			izz="0.1"
+		/>
+		</inertial>
+		<collision name="left_wheel_collision">
+			<origin xyz="0 0 0" rpy="0 1.5707 1.5707"/>
+			<geometry>
+				<cylinder radius="0.1" length="0.05"/>
+			</geometry>
+		</collision>
+		<visual name="left_wheel_visual">
+			<origin xyz="0 0 0" rpy="0 1.5707 1.5707"/>
+			<geometry>
+				<cylinder radius="0.1" length="0.05"/>
+			</geometry>
+		</visual>
+	</link>
+	<link name="right_wheel">
+		<inertial>
+		<mass value="5.0"/>
+		<origin xyz="0 0 0" rpy="0 1.5707 1.5707"/>
+		<inertia
+			ixx="0.1" ixy="0" ixz="0"
+			iyy="0.1" iyz="0"
+			izz="0.1"
+		/>
+		</inertial>
+		<collision name="right_wheel_collision">
+			<origin xyz="0 0 0" rpy="0 1.5707 1.5707"/>
+			<geometry>
+				<cylinder radius="0.1" length="0.05"/>
+			</geometry>
+		</collision>
+		<visual name="right_wheel_visual">
+			<origin xyz="0 0 0" rpy="0 1.5707 1.5707"/>
+			<geometry>
+				<cylinder radius="0.1" length="0.05"/>
+			</geometry>
+		</visual>
+	</link>
+	<joint type="continuous" name="left_wheel_hinge">
+		<origin xyz="0 0.15 0" rpy="0 0 0"/>
+		<child link="left_wheel"/>
+		<parent link="chassis"/>
+		<axis xyz="0 1 0" rpy="0 0 0"/>
+		<limit effort="10000" velocity="1000"/>
+		<dynamics damping="1.0" friction="1.0"/>
+	</joint>
+	<joint type="continuous" name="right_wheel_hinge">
+		<origin xyz="0 -0.15 0" rpy="0 0 0"/>
+		<child link="right_wheel"/>
+		<parent link="chassis"/>
+		<axis xyz="0 1 0" rpy="0 0 0"/>
+		<limit effort="10000" velocity="1000"/>
+		<dynamics damping="1.0" friction="1.0"/>
+	</joint>
+	<link name="camera">
+		<inertial>
+		<mass value="0.1"/>
+		<origin xyz="0 0 0" rpy="0 0 0"/>
+		<inertia
+			ixx="1e-6" ixy="0" ixz="0"
+			iyy="1e-6" iyz="0"
+			izz="1e-6"/>
+		</inertial>
+		<collision name="camera_collision">
+			<origin xyz="0 0 0" rpy="0 0 0"/>
+			<geometry>
+				<box size="0.05 0.05 0.05"/>
+			</geometry>
+		</collision>
+		<visual name="camera_visual">
+			<origin xyz="0 0 0" rpy="0 0 0"/>
+			<geometry>
+				<box size="0.05 0.05 0.05"/>
+			</geometry>
+		</visual>
+	</link>
+	<joint name="camera_joint" type="fixed">
+		<axis xyz="0 1 0"/>
+		<origin xyz="0.2 0 0" rpy="0 0 0"/>
+		<parent link = "chassis"/>
+		<child link="camera"/>
+	</joint>
+	<link name="hokuyo">
+		<inertial>
+		<mass value="1e-5"/>
+		<origin xyz="0 0 0" rpy="0 0 0"/>
+		<inertia
+			ixx="1e-6" ixy="0" ixz="0"
+			iyy="1e-6" iyz="0"
+			izz="1e-6"/>
+		</inertial>
+		<collision name="hokuyo_collision">
+			<origin xyz="0 0 0" rpy="0 0 0"/>
+			<geometry>
+				<box size="0.1 0.1 0.1"/>
+			</geometry>
+		</collision>
+		<visual name="hokuyo_visual">
+			<origin xyz="0 0 0" rpy="0 0 0"/>
+			<geometry>
+				<mesh filename="package://my_robot/meshes/hokuyo.dae"/>
+			</geometry>
+		</visual>
+	</link>
+	<joint name="hokuyo_joint" type="fixed">
+		<axis xyz="0 1 0"/>
+		<origin xyz="0.15 0 0.1" rpy="0 0 0"/>
+		<parent link = "chassis"/>
+		<child link="hokuyo"/>
+	</joint>
+	<gazebo reference="chassis">
+		<material>Gazebo/Blue</material>
+	</gazebo>
+	<gazebo reference="left_wheel">
+		<material>Gazebo/Green</material>
+	</gazebo>
+	<gazebo reference="right_wheel">
+		<material>Gazebo/Green</material>
+	</gazebo>
+	<gazebo reference="camera">
+		<material>Gazebo/Red</material>
+	</gazebo>
+	<gazebo reference="chassis">
+		<material>Gazebo/Blue</material>
+	</gazebo>
 </robot>

Commit message: Trying to create a plugin for Gazebo

File: catkin_ws/src/my_robot/urdf/my_robot.xacro (robot description, xacro)
@@ -9,5 +9,5 @@
 	</joint>
 	<link name="chassis">
-		<pose>0 0 0.1 0 0 0</pose>
+		<pose>0 0 0.5 0 0 0</pose>
 	<inertial>
 		<mass value="15.0"/>
@@ -19,8 +19,8 @@
 		/>
 	</inertial>
-	<collision name="collision">
+	<collision name="chassis_collision">
 		<origin xyz="0 0 0" rpy=" 0 0 0"/>
 		<geometry>
-			<box size=".4 .2 .1"/>
+			<cylinder length="0.1" radius="0.3"/>
 		</geometry>
 	</collision>
@@ -28,5 +28,5 @@
 		<origin xyz="0 0 0" rpy=" 0 0 0"/>
 		<geometry>
-			<box size=".4 .2 .1"/>
+			<cylinder length="0.1" radius="0.3"/>
 		</geometry>
 	</visual>
@@ -142,5 +142,5 @@
 	<joint name="camera_joint" type="fixed">
 		<axis xyz="0 1 0"/>
-		<origin xyz="0.2 0 0" rpy="0 0 0"/>
+		<origin xyz="0.3 0 0" rpy="0 0 0"/>
 		<parent link = "chassis"/>
 		<child link="camera"/>
@@ -170,5 +170,5 @@
 	<joint name="hokuyo_joint" type="fixed">
 		<axis xyz="0 1 0"/>
-		<origin xyz="0.15 0 0.1" rpy="0 0 0"/>
+		<origin xyz="0.15 0 0.08" rpy="0 0 0"/>
 		<parent link = "chassis"/>
 		<child link="hokuyo"/>

Commit message: Updated files for contact sensor

File: catkin_ws/src/my_robot/urdf/my_robot.xacro (robot description, xacro)
@@ -56,4 +56,29 @@
 	</visual>
 	</link>
+	<link name="bump_sensor">
+		<collision name="bump_sensor_collision">
+		<origin xyz="0 0 0" rpy="0 0 0"/>
+		<geometry>
+		<box size="0.065 1.0 0.02"/>
+		</geometry>
+		</collision>
+		 <visual>
+      			<origin xyz="0 0 0" rpy="0 0 0"/>
+      			<geometry>
+         			<box size="0.065 1.0 0.02"/>
+      			</geometry>
+    		</visual>
+    		<inertial>
+      			<mass value="1e-5" />
+      			<origin xyz="0 0 0" rpy="0 0 0"/>
+      		<inertia ixx="1e-6" ixy="0" ixz="0" iyy="1e-6" iyz="0" izz="1e-6" />
+    		</inertial>
+  	</link>
+	<joint name="bumper_joint" type="fixed">
+		<axis xyz="0 1 0"/>
+		<origin xyz="0.3 0 -0.05" rpy="0 0 0"/>
+		<parent link="chassis"/>
+		<child link="bump_sensor"/>
+	</joint>
 	<link name="left_wheel">
 		<inertial>
@@ -189,3 +214,6 @@
 		<material>Gazebo/Blue</material>
 	</gazebo>
+	<gazebo reference="bump_sensor">
+		<material>Gazebo/Black</material>
+	</gazebo>
 </robot>
